File: trim_relay.sch (KiCad schematic (older format))
At the start: 29 parts, among them J1 Conn_01x01, J10 Conn_01x01, J11 Conn_01x01, J12 Conn_01x01, J13 GS2, J14 GS2, J2 Conn_01x01, J3 Conn_01x01, J4 Conn_01x01, J5 Conn_01x01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

Commit message: new version kicad changes
Parts:
- C1, C2: symbol CP -> trim_relay-rescue:CP
- D1, D2, D3, D4, D5: symbol D -> trim_relay-rescue:D
- J1, J10, J11, J12, J2, J3, J4, J5, J6, J7, J8, J9: symbol Conn_01x01 -> trim_relay-rescue:Conn_01x01
- J13, J14: symbol GS2 -> trim_relay-rescue:GS2
- K1, K2, K3, K4, K5: symbol G5Q-1 -> trim_relay-rescue:G5Q-1
- R7: symbol R -> trim_relay-rescue:R
- RV1: symbol POT -> trim_relay-rescue:POT
- U1: symbol LM317L_TO92 -> trim_relay-rescue:LM317L_TO92
